Commit message: second commit

File: description/robot.urdf.xacro (robot description, xacro)
@@ -2,3 +2,4 @@
 <robot xmlns:xacro="http://www.ros.org/wiki/xacro"  name="robot">
     <xacro:include filename="robot_core.xacro" />
+    <xacro:include filename="gazebo_control.xacro"/>
 </robot>

File: description/robot_core.xacro (robot description, xacro)
@@ -2,4 +2,5 @@
 <robot xmlns:xacro="http://www.ros.org/wiki/xacro" >
     <xacro:include filename="inertial_macros.xacro"/>
+    <xacro:include filename="gazebo_control.xacro"/>
     <material name="white">
         <color rgba="1 1 1 1" />
@@ -41,4 +42,7 @@
         </xacro:inertial_box>
     </link>
+    <gazebo reference="chassis_link">
+        <material>Gazebo/White</material>
+    </gazebo>
     <!-- left wheel Link -->
     <joint name="leftwheel_joint" type="continuous">
@@ -66,4 +70,7 @@
         </xacro:inertial_cylinder>
     </link>
+    <gazebo reference="leftwheel_link">
+        <material>Gazebo/Blue</material>
+    </gazebo>
     <!-- right wheel Link -->
     <joint name="rightwheel_joint" type="continuous">
@@ -91,4 +98,7 @@
         </xacro:inertial_cylinder>
     </link>
+    <gazebo reference="rightwheel_link">
+        <material>Gazebo/Blue</material>
+    </gazebo>
     <!-- Caster wheel link-->
     <joint name="casterwheel_joint" type="fixed">
@@ -115,3 +125,8 @@
         </xacro:inertial_sphere>
     </link>
+    <gazebo reference="casterwheel_link">
+        <material>Gazebo/Black</material>
+        <mu1 value="0.001"/>
+        <mu2 value="0.001"/>
+    </gazebo>
 </robot>
